File: Alimentacion.kicad_sch (KiCad schematic)
At the start: 0 parts

Commit message: Alimentación
Parts:
- added C5: 0.01uF, Samacsys:1366004, symbol Device:C
- added C6: 1uF, Samacsys:1366004, symbol Device:C
- added C7: 10uF, Samacsys:1366004, symbol Device:C
- added J1: 1366004, Samacsys:1366004, symbol Samacsys:1366004
- added PS1: TAR5SB30_TE85L,F_, Samacsys:SOT95P275X140-5N, symbol Samacsys:TAR5SB30_TE85L,F_
Connections:
- net Vout3v: now also C7.1, PS1.5 (VOUT)
- new net: C5.1, PS1.4 (NOISE)
- new net +9V: C6.1, J1.1, PS1.1 (VIN), PS1.3 (CONTROL)
- new net GND: C5.2, C6.2, C7.2, J1.2, PS1.2 (GND)

Commit message: Ejercicio practico clase 3
Parts:
- C1: renamed from C6; footprint Samacsys:1366004 -> Capacitor_SMD:C_0402_1005Metric
- C2: renamed from C5; footprint Samacsys:1366004 -> Capacitor_SMD:C_0402_1005Metric
- C3: renamed from C7; footprint Samacsys:1366004 -> Capacitor_SMD:C_0402_1005Metric
Connections:
- no-connect marks 0 -> 2
Changed lines of the file:
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@@
 	(paper "A4")
+	(junction
+		(at 41.91 88.9)
+		(diameter 0)
+		(color 0 0 0 0)
+	)
+	(junction
+		(at 33.02 85.09)
+		(diameter 0)
+		(color 0 0 0 0)
+	)
 	(junction
 		(at 39.37 85.09)
@@
 		(color 0 0 0 0)
 	)
+	(no_connect
+		(at 64.77 87.63)
+	)
+	(no_connect
+		(at 64.77 85.09)
+	)
 	(wire
 		(pts
@@
 	(wire
 		(pts
+			(xy 29.21 82.55) (xy 29.21 85.09)
+		)
+		(stroke
+			(width 0)
+			(type default)
+		)
+	)
+	(wire
+		(pts
 			(xy 74.93 85.09) (xy 74.93 72.39)
 		)
@@
 	(wire
 		(pts
+			(xy 29.21 85.09) (xy 33.02 85.09)
+		)
+		(stroke
+			(width 0)
+			(type default)
+		)
+	)
+	(wire
+		(pts
+			(xy 36.83 88.9) (xy 41.91 88.9)
+		)
+		(stroke
+			(width 0)
+			(type default)
+		)
+	)
+	(wire
+		(pts
 			(xy 152.4 87.63) (xy 154.94 87.63)
 		)
@@
 	(wire
 		(pts
-			(xy 41.91 87.63) (xy 41.91 91.44)
+			(xy 41.91 87.63) (xy 41.91 88.9)
 		)
 		(stroke
@@
 		(pts
 			(xy 156.21 74.93) (xy 156.21 85.09)
+		)
+		(stroke
+			(width 0)
+			(type default)
+		)
+	)
+	(wire
+		(pts
+			(xy 41.91 88.9) (xy 41.91 91.44)
 		)
 		(stroke
@@
 	)
 	(symbol
+		(lib_id "power:PWR_FLAG")
+		(at 36.83 88.9 0)
+		(mirror y)
+		(unit 1)
+		(body_style 1)
+		(exclude_from_sim no)
+		(in_bom yes)
+		(on_board yes)
+		(in_pos_files yes)
+		(dnp no)
+		(property "Reference" "#FLG02"
+			(at 36.83 86.995 0)
+			(hide yes)
+			(show_name no)
+			(do_not_autoplace no)
+			(effects
+				(font
+					(size 1.27 1.27)
+				)
+			)
+		)
+		(property "Value" "PWR_FLAG"
+			(at 35.814 90.424 0)
+			(show_name no)
+			(do_not_autoplace no)
+			(effects
+				(font
+					(size 1.27 1.27)
+				)
+			)
+		)
+		(property "Footprint" "Package_DIP:DIP-24_W7.62mm"
+			(at 36.83 88.9 0)
+			(hide yes)
+			(show_name no)
+			(do_not_autoplace no)
+			(effects
+				(font
+					(size 1.27 1.27)
+				)
+			)
+		)
+		(property "Datasheet" ""
+			(at 36.83 88.9 0)
+			(hide yes)
+			(show_name no)
+			(do_not_autoplace no)
+			(effects
+				(font
+					(size 1.27 1.27)
+				)
+			)
+		)
+		(property "Description" "Special symbol for telling ERC where power comes from"
+			(at 36.83 88.9 0)
+			(hide yes)
+			(show_name no)
+			(do_not_autoplace no)
+			(effects
+				(font
+					(size 1.27 1.27)
+				)
+			)
+		)
+		(pin "1"
+		)
+		(instances
+			(project "sesion2"
+				(path "/d1e9e723-5327-48d1-b5e7-0bbac6992fdf/c1caa85c-9bda-46ac-bb58-ca6470d629ed"
+					(reference "#FLG02")
+					(unit 1)
+				)
+			)
+		)
+	)
+	(symbol
+		(lib_id "power:PWR_FLAG")
+		(at 29.21 82.55 0)
+		(mirror y)
+		(unit 1)
+		(body_style 1)
+		(exclude_from_sim no)
+		(in_bom yes)
+		(on_board yes)
+		(in_pos_files yes)
+		(dnp no)
+		(property "Reference" "#FLG01"
+			(at 29.21 80.645 0)
+			(hide yes)
+			(show_name no)
+			(do_not_autoplace no)
+			(effects
+				(font
+					(size 1.27 1.27)
+				)
+			)
+		)
+		(property "Value" "PWR_FLAG"
+			(at 23.876 82.55 0)
+			(show_name no)
+			(do_not_autoplace no)
+			(effects
+				(font
+					(size 1.27 1.27)
+				)
+			)
+		)
+		(property "Footprint" "Package_DIP:DIP-24_W7.62mm"
+			(at 29.21 82.55 0)
+			(hide yes)
+			(show_name no)
+			(do_not_autoplace no)
+			(effects
+				(font
+					(size 1.27 1.27)
+				)
+			)
+		)
+		(property "Datasheet" ""
+			(at 29.21 82.55 0)
+			(hide yes)
+			(show_name no)
+			(do_not_autoplace no)
+			(effects
+				(font
+					(size 1.27 1.27)
+				)
+			)
+		)
+		(property "Description" "Special symbol for telling ERC where power comes from"
+			(at 29.21 82.55 0)
+			(hide yes)
+			(show_name no)
+			(do_not_autoplace no)
+			(effects
+				(font
+					(size 1.27 1.27)
+				)
+			)
+		)
+		(pin "1"
+		)
+		(instances
+			(project "sesion2"
+				(path "/d1e9e723-5327-48d1-b5e7-0bbac6992fdf/c1caa85c-9bda-46ac-bb58-ca6470d629ed"
+					(reference "#FLG01")
+					(unit 1)
+				)
+			)
+		)
+	)
+	(symbol
 		(lib_id "Device:C")
 		(at 156.21 71.12 180)
@@
 		(dnp no)
 		(fields_autoplaced yes)
-		(property "Reference" "C5"
+		(property "Reference" "C2"
 			(at 160.02 69.8499 0)
 			(show_name no)
@@
 			)
 		)
-		(property "Footprint" "Samacsys:1366004"
+		(property "Footprint" "Capacitor_SMD:C_0402_1005Metric"
 			(at 155.2448 67.31 0)
 			(hide yes)
@@
 			(project "sesion2"
 				(path "/d1e9e723-5327-48d1-b5e7-0bbac6992fdf/c1caa85c-9bda-46ac-bb58-ca6470d629ed"
-					(reference "C5")
+					(reference "C2")
 					(unit 1)
 				)
@@
 		(dnp no)
 		(fields_autoplaced yes)
-		(property "Reference" "C6"
+		(property "Reference" "C1"
 			(at 114.3 73.66 90)
 			(show_name no)
@@
 			)
 		)
-		(property "Footprint" "Samacsys:1366004"
+		(property "Footprint" "Capacitor_SMD:C_0402_1005Metric"
 			(at 110.49 82.2452 0)
 			(hide yes)
@@
 			(project "sesion2"
 				(path "/d1e9e723-5327-48d1-b5e7-0bbac6992fdf/c1caa85c-9bda-46ac-bb58-ca6470d629ed"
-					(reference "C6")
+					(reference "C1")
 					(unit 1)
 				)
@@
 		(in_pos_files yes)
 		(dnp no)
-		(property "Reference" "C7"
+		(property "Reference" "C3"
 			(at 158.75 100.33 90)
 			(show_name no)
@@
 			)
 		)
-		(property "Footprint" "Samacsys:1366004"
+		(property "Footprint" "Capacitor_SMD:C_0402_1005Metric"
 			(at 162.56 94.2848 0)
 			(hide yes)
@@
 			(project "sesion2"
 				(path "/d1e9e723-5327-48d1-b5e7-0bbac6992fdf/c1caa85c-9bda-46ac-bb58-ca6470d629ed"
-					(reference "C7")
+					(reference "C3")
 					(unit 1)
 				)
@@
 		(dnp no)
 		(fields_autoplaced yes)
-		(property "Reference" "#PWR04"
+		(property "Reference" "#PWR02"
 			(at 41.91 97.79 0)
 			(hide yes)
@@
 			(project "sesion2"
 				(path "/d1e9e723-5327-48d1-b5e7-0bbac6992fdf/c1caa85c-9bda-46ac-bb58-ca6470d629ed"
-					(reference "#PWR04")
+					(reference "#PWR02")
 					(unit 1)
 				)
@@
 		(dnp no)
 		(fields_autoplaced yes)
-		(property "Reference" "#PWR03"
+		(property "Reference" "#PWR05"
 			(at 156.21 60.96 0)
 			(hide yes)
@@
 			(project "sesion2"
 				(path "/d1e9e723-5327-48d1-b5e7-0bbac6992fdf/c1caa85c-9bda-46ac-bb58-ca6470d629ed"
-					(reference "#PWR03")
+					(reference "#PWR05")
 					(unit 1)
 				)
@@
 		(dnp no)
 		(fields_autoplaced yes)
-		(property "Reference" "#PWR06"
+		(property "Reference" "#PWR03"
 			(at 99.06 81.28 0)
 			(hide yes)
@@
 			(project "sesion2"
 				(path "/d1e9e723-5327-48d1-b5e7-0bbac6992fdf/c1caa85c-9bda-46ac-bb58-ca6470d629ed"
-					(reference "#PWR06")
+					(reference "#PWR03")
 					(unit 1)
 				)
@@
 		(dnp no)
 		(fields_autoplaced yes)
-		(property "Reference" "#PWR07"
+		(property "Reference" "#PWR06"
 			(at 173.99 95.25 0)
 			(hide yes)
@@
 			(project "sesion2"
 				(path "/d1e9e723-5327-48d1-b5e7-0bbac6992fdf/c1caa85c-9bda-46ac-bb58-ca6470d629ed"
-					(reference "#PWR07")
+					(reference "#PWR06")
 					(unit 1)
 				)
@@
 		(dnp no)
 		(fields_autoplaced yes)
-		(property "Reference" "#PWR02"
+		(property "Reference" "#PWR04"
 			(at 105.41 87.63 0)
 			(hide yes)
@@
 			(project "sesion2"
 				(path "/d1e9e723-5327-48d1-b5e7-0bbac6992fdf/c1caa85c-9bda-46ac-bb58-ca6470d629ed"
-					(reference "#PWR02")
+					(reference "#PWR04")
 					(unit 1)
 				)

Commit message: sesion 4
Parts:
- removed C1: 1uF, Capacitor_SMD:C_0402_1005Metric, symbol Device:C
- removed C2: 0.01uF, Capacitor_SMD:C_0402_1005Metric, symbol Device:C
- removed C3: 10uF, Capacitor_SMD:C_0402_1005Metric, symbol Device:C
- removed J1: 1366004, Samacsys:1366004, symbol Samacsys:1366004
- removed PS1: TAR5SB30_TE85L,F_, Samacsys:SOT95P275X140-5N, symbol Samacsys:TAR5SB30_TE85L,F_
- added CCOMP1: 82 nF, Capacitor_SMD:C_0402_1005Metric, symbol Device:C
- added CCOMP2: 180pF, Capacitor_SMD:C_0402_1005Metric, symbol Device:C
- added Cboot1: 100 nF, Capacitor_SMD:C_0402_1005Metric, symbol Device:C
- added Cin1, Cin2: 4.7 uF, Capacitor_SMD:C_0402_1005Metric, symbol Device:C
- added Cout1, Cout2: 22 uF, Capacitor_SMD:C_0402_1005Metric, symbol Device:C
- added D1: B560C, Samacsys:DIOM7959X250N, symbol Samacsys:B560C
- added J1: TB0012-508-02GR, Samacsys:TB0012-508-02GR, symbol Samacsys:TB0012-508-02GR
- added L1: 10uH, Inductor_SMD:L_1206_3216Metric, symbol Device:L
- added RCOMP1: 3.24, Resistor_SMD:R_0402_1005Metric_Pad0.72x0.64mm_HandSolder, symbol Device:R
- added REN1: 100k, Resistor_SMD:R_0402_1005Metric_Pad0.72x0.64mm_HandSolder, symbol Device:R
- added REN2, RFB2: 10k, Resistor_SMD:R_0402_1005Metric_Pad0.72x0.64mm_HandSolder, symbol Device:R
- added RFB1: 31.2k, Resistor_SMD:R_0402_1005Metric_Pad0.72x0.64mm_HandSolder, symbol Device:R
- added RRT1: 340k, Resistor_SMD:R_0402_1005Metric_Pad0.72x0.64mm_HandSolder, symbol Device:R
- added U1: TPS54360BDDA, Samacsys:SOIC127P600X170-9N, symbol Samacsys:TPS54360BDDA
Connections:
- net GND: now also CCOMP1.2, CCOMP2.2, Cin1.2, Cin2.2, Cout1.2, Cout2.2, D1.2 (A), J1.2, REN2.2, RFB2.2, RRT1.2, U1.7 (GND), U1.9 (EP)
- new net: CCOMP2.1, RCOMP1.1, U1.6 (COMP)
- new net: RRT1.1, U1.4 (RT/CLK)
- new net: Cboot1.1, U1.1 (BOOT)
- new net: Cin1.1, Cin2.1, J1.1, REN1.1, U1.2 (VIN)
- new net: REN1.2, REN2.1, U1.3 (EN)
- new net: Cboot1.2, D1.1 (K), L1.1, U1.8 (SW)
- new net: CCOMP1.1, RCOMP1.2
- new net 3.3v: Cout1.1, Cout2.1, L1.2, RFB1.1
- new net FB: RFB1.2, RFB2.1, U1.5 (FB)
- no-connect marks 2 -> 0

Commit message: Se han implementado componentes de protección en las líneas de entrada
Parts:
- added D2: D_TVS, Diode_SMD:D_SMA, symbol Device:D_TVS
- added TP1: TestPoint, TestPoint:TestPoint_Pad_1.5x1.5mm, symbol Connector:TestPoint
Connections:
- net 3.3v: now also TP1.1
- net GND: now also D2.2 (A2)
- net at Cin1.1, Cin2.1, J1.1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: now also D2.1 (A1)
Other:
- moved on the sheet: Cin1, Cin2
Changed lines of the file:
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@@
 	(paper "A4")
 	(junction
-		(at 76.2 130.81)
+		(at 77.47 130.81)
 		(diameter 0)
 		(color 0 0 0 0)
@@
 	)
 	(junction
-		(at 82.55 130.81)
+		(at 83.82 130.81)
 		(diameter 0)
 		(color 0 0 0 0)
@@
 	)
 	(junction
+		(at 73.66 99.06)
+		(diameter 0)
+		(color 0 0 0 0)
+	)
+	(junction
+		(at 71.12 106.68)
+		(diameter 0)
+		(color 0 0 0 0)
+	)
+	(junction
 		(at 143.51 130.81)
 		(diameter 0)
@@
 	)
 	(junction
+		(at 217.17 80.01)
+		(diameter 0)
+		(color 0 0 0 0)
+	)
+	(junction
 		(at 125.73 130.81)
 		(diameter 0)
@@
 	)
 	(junction
-		(at 82.55 99.06)
+		(at 83.82 99.06)
 		(diameter 0)
 		(color 0 0 0 0)
@@
 	)
 	(junction
-		(at 76.2 99.06)
+		(at 77.47 99.06)
 		(diameter 0)
 		(color 0 0 0 0)
@@
 	(wire
 		(pts
-			(xy 76.2 106.68) (xy 76.2 99.06)
+			(xy 77.47 106.68) (xy 77.47 99.06)
 		)
 		(stroke
@@
 	(wire
 		(pts
-			(xy 71.12 99.06) (xy 76.2 99.06)
+			(xy 71.12 99.06) (xy 73.66 99.06)
 		)
 		(stroke
@@
 	(wire
 		(pts
-			(xy 76.2 99.06) (xy 82.55 99.06)
-		)
-		(stroke
-			(width 0)
-			(type default)
-		)
-	)
-	(wire
-		(pts
-			(xy 71.12 130.81) (xy 76.2 130.81)
+			(xy 71.12 130.81) (xy 86.36 130.81)
 		)
 		(stroke
@@
 	(wire
 		(pts
+			(xy 71.12 106.68) (xy 73.66 106.68)
+		)
+		(stroke
+			(width 0)
+			(type default)
+		)
+	)
+	(wire
+		(pts
 			(xy 193.04 95.25) (xy 193.04 99.06)
 		)
@@
 	(wire
 		(pts
-			(xy 82.55 99.06) (xy 101.6 99.06)
-		)
-		(stroke
-			(width 0)
-			(type default)
-		)
-	)
-	(wire
-		(pts
-			(xy 82.55 99.06) (xy 82.55 106.68)
+			(xy 83.82 99.06) (xy 83.82 106.68)
 		)
 		(stroke
@@
 	(wire
 		(pts
-			(xy 76.2 130.81) (xy 82.55 130.81)
-		)
-		(stroke
-			(width 0)
-			(type default)
-		)
-	)
-	(wire
-		(pts
-			(xy 71.12 101.6) (xy 71.12 130.81)
+			(xy 71.12 101.6) (xy 71.12 106.68)
 		)
 		(stroke
@@
 	(wire
 		(pts
-			(xy 82.55 114.3) (xy 82.55 130.81)
+			(xy 83.82 114.3) (xy 83.82 130.81)
 		)
 		(stroke
@@
 	(wire
 		(pts
+			(xy 73.66 99.06) (xy 101.6 99.06)
+		)
+		(stroke
+			(width 0)
+			(type default)
+		)
+	)
+	(wire
+		(pts
 			(xy 96.52 130.81) (xy 96.52 133.35)
 		)
@@
 	(wire
 		(pts
+			(xy 217.17 80.01) (xy 222.25 80.01)
+		)
+		(stroke
+			(width 0)
+			(type default)
+		)
+	)
+	(wire
+		(pts
 			(xy 101.6 99.06) (xy 128.27 99.06)
 		)
@@
 	(wire
 		(pts
+			(xy 71.12 106.68) (xy 71.12 130.81)
+		)
+		(stroke
+			(width 0)
+			(type default)
+		)
+	)
+	(wire
+		(pts
 			(xy 167.64 101.6) (xy 179.07 101.6)
 		)
@@
 	(wire
 		(pts
-			(xy 76.2 114.3) (xy 76.2 130.81)
-		)
-		(stroke
-			(width 0)
-			(type default)
-		)
-	)
-	(wire
-		(pts
-			(xy 82.55 130.81) (xy 86.36 130.81)
-		)
-		(stroke
-			(width 0)
-			(type default)
-		)
-	)
-	(wire
-		(pts
-			(xy 210.82 80.01) (xy 222.25 80.01)
+			(xy 77.47 114.3) (xy 77.47 130.81)
+		)
+		(stroke
+			(width 0)
+			(type default)
+		)
+	)
+	(wire
+		(pts
+			(xy 210.82 80.01) (xy 217.17 80.01)
 		)
 		(stroke
@@
 				(path "/d1e9e723-5327-48d1-b5e7-0bbac6992fdf/c1caa85c-9bda-46ac-bb58-ca6470d629ed"
 					(reference "CCOMP2")
+					(unit 1)
+				)
+			)
+		)
+	)
+	(symbol
+		(lib_id "Device:D_TVS")
+		(at 73.66 102.87 270)
+		(unit 1)
+		(body_style 1)
+		(exclude_from_sim no)
+		(in_bom yes)
+		(on_board yes)
+		(in_pos_files yes)
+		(dnp no)
+		(fields_autoplaced yes)
+		(property "Reference" "D2"
+			(at 76.2 101.5999 90)
+			(show_name no)
+			(do_not_autoplace no)
+			(effects
+				(font
+					(size 1.27 1.27)
+				)
+				(justify left)
+			)
+		)
+		(property "Value" "D_TVS"
+			(at 76.2 104.1399 90)
+			(show_name no)
+			(do_not_autoplace no)
+			(effects
+				(font
+					(size 1.27 1.27)
+				)
+				(justify left)
+			)
+		)
+		(property "Footprint" "Diode_SMD:D_SMA"
+			(at 73.66 102.87 0)
+			(hide yes)
+			(show_name no)
+			(do_not_autoplace no)
+			(effects
+				(font
+					(size 1.27 1.27)
+				)
+			)
+		)
+		(property "Datasheet" ""
+			(at 73.66 102.87 0)
+			(hide yes)
+			(show_name no)
+			(do_not_autoplace no)
+			(effects
+				(font
+					(size 1.27 1.27)
+				)
+			)
+		)
+		(property "Description" "Bidirectional transient-voltage-suppression diode"
+			(at 73.66 102.87 0)
+			(hide yes)
+			(show_name no)
+			(do_not_autoplace no)
+			(effects
+				(font
+					(size 1.27 1.27)
+				)
+			)
+		)
+		(pin "2"
+		)
+		(pin "1"
+		)
+		(instances
+			(project "sesion2"
+				(path "/d1e9e723-5327-48d1-b5e7-0bbac6992fdf/c1caa85c-9bda-46ac-bb58-ca6470d629ed"
+					(reference "D2")
+					(unit 1)
+				)
+			)
+		)
+	)
+	(symbol
+		(lib_id "Connector:TestPoint")
+		(at 217.17 80.01 0)
+		(unit 1)
+		(body_style 1)
+		(exclude_from_sim no)
+		(in_bom yes)
+		(on_board yes)
+		(in_pos_files yes)
+		(dnp no)
+		(fields_autoplaced yes)
+		(property "Reference" "TP1"
+			(at 219.71 75.4379 0)
+			(show_name no)
+			(do_not_autoplace no)
+			(effects
+				(font
+					(size 1.27 1.27)
+				)
+				(justify left)
+			)
+		)
+		(property "Value" "TestPoint"
+			(at 219.71 77.9779 0)
+			(show_name no)
+			(do_not_autoplace no)
+			(effects
+				(font
+					(size 1.27 1.27)
+				)
+				(justify left)
+			)
+		)
+		(property "Footprint" "TestPoint:TestPoint_Pad_1.5x1.5mm"
+			(at 222.25 80.01 0)
+			(hide yes)
+			(show_name no)
+			(do_not_autoplace no)
+			(effects
+				(font
+					(size 1.27 1.27)
+				)
+			)
+		)
+		(property "Datasheet" ""
+			(at 222.25 80.01 0)
+			(hide yes)
+			(show_name no)
+			(do_not_autoplace no)
+			(effects
+				(font
+					(size 1.27 1.27)
+				)
+			)
+		)
+		(property "Description" "test point"
+			(at 217.17 80.01 0)
+			(hide yes)
+			(show_name no)
+			(do_not_autoplace no)
+			(effects
+				(font
+					(size 1.27 1.27)
+				)
+			)
+		)
+		(pin "1"
+		)
+		(instances
+			(project "sesion2"
+				(path "/d1e9e723-5327-48d1-b5e7-0bbac6992fdf/c1caa85c-9bda-46ac-bb58-ca6470d629ed"
+					(reference "TP1")
 					(unit 1)
 				)
@@
 	(symbol
 		(lib_id "Device:C")
-		(at 76.2 110.49 0)
+		(at 77.47 110.49 0)
 		(unit 1)
 		(body_style 1)
@@
 		(dnp no)
 		(property "Reference" "Cin1"
-			(at 73.406 108.458 0)
+			(at 74.676 108.458 0)
 			(show_name no)
 			(do_not_autoplace no)
@@
 		)
 		(property "Value" "4.7 uF"
-			(at 72.39 113.03 0)
+			(at 73.66 113.03 0)
 			(show_name no)
 			(do_not_autoplace no)
@@
 		)
 		(property "Footprint" "Capacitor_SMD:C_0402_1005Metric"
-			(at 77.1652 114.3 0)
+			(at 78.4352 114.3 0)
 			(hide yes)
 			(show_name no)
@@
 		)
 		(property "Datasheet" ""
-			(at 76.2 110.49 0)
+			(at 77.47 110.49 0)
 			(hide yes)
 			(show_name no)
@@
 		)
 		(property "Description" "Unpolarized capacitor"
-			(at 76.2 110.49 0)
+			(at 77.47 110.49 0)
 			(hide yes)
 			(show_name no)
@@
 	(symbol
 		(lib_id "Device:C")
-		(at 82.55 110.49 0)
+		(at 83.82 110.49 0)
 		(unit 1)
 		(body_style 1)
@@
 		(dnp no)
 		(property "Reference" "Cin2"
-			(at 83.82 108.458 0)
+			(at 85.09 108.458 0)
 			(show_name no)
 			(do_not_autoplace no)
@@
 		)
 		(property "Value" "4.7 uF"
-			(at 83.82 113.03 0)
+			(at 85.09 113.03 0)
 			(show_name no)
 			(do_not_autoplace no)
@@
 		)
 		(property "Footprint" "Capacitor_SMD:C_0402_1005Metric"
-			(at 83.5152 114.3 0)
+			(at 84.7852 114.3 0)
 			(hide yes)
 			(show_name no)
@@
 		)
 		(property "Datasheet" ""
-			(at 82.55 110.49 0)
+			(at 83.82 110.49 0)
 			(hide yes)
 			(show_name no)
@@
 		)
 		(property "Description" "Unpolarized capacitor"
-			(at 82.55 110.49 0)
-			(hide yes)
-			(show_name no)
+			(at 83.82 110.49 0)
+			(hide yes)
+			(show_name no)
