File: Microcontrolador.kicad_sch (KiCad schematic)
At the start: 6 parts

Commit message: Esquematico microcontrolador
Parts:
- added IC1: AT89LS51-16AU, Samacsys:QFP80P1200X1200X120-44N, symbol Samacsys:AT89LS51-16AU
- added J1: 68000-106HLF, Samacsys:HDRV6W64P0X254_1X6_1524X254X839P, symbol Samacsys:68000-106HLF
Connections:
- net vdd_mcu: now also IC1.38 (VCC), J1.1
- net at R1.1: now also J1.4
- net at C1.1, R1.2: now also IC1.41 (P1.1)
- net at C3.1, R3.2: now also IC1.40 (P1.0)
- net GND: now reaches C3.2
- net GND: now also C1.2, C2.2, IC1.16 (GND_1), J1.2
- net at C2.1, R2.2: now also IC1.42 (P1.2)
- net at R3.1: now also J1.5
- net at R2.1: now also J1.3
- no-connect marks 0 -> 40
Other:
- moved on the sheet: C1, C2, C3, R1, R2, R3

Commit message: Ejercicio practico clase 3
Parts:
- added C7: 100nF, Capacitor_SMD:C_0402_1005Metric, symbol Device:C
- C4: renamed from C2; footprint Samacsys:HDRV6W64P0X254_1X6_1524X254X839P -> Capacitor_SMD:C_0402_1005Metric
- C5: renamed from C1; footprint Samacsys:HDRV6W64P0X254_1X6_1524X254X839P -> Capacitor_SMD:C_0402_1005Metric
- C6: renamed from C3; footprint Samacsys:HDRV6W64P0X254_1X6_1524X254X839P -> Capacitor_SMD:C_0402_1005Metric
- R1: renamed from R2; footprint Package_LCC:PLCC-84_29.3x29.3mm_P1.27mm -> Resistor_SMD:R_0402_1005Metric_Pad0.72x0.64mm_HandSolder
- R2: renamed from R1; footprint Package_LCC:PLCC-84_29.3x29.3mm_P1.27mm -> Resistor_SMD:R_0402_1005Metric_Pad0.72x0.64mm_HandSolder
- R3: footprint Package_LCC:PLCC-84_29.3x29.3mm_P1.27mm -> Resistor_SMD:R_0402_1005Metric_Pad0.72x0.64mm_HandSolder
- renumbered J1 to J2
Connections:
- net GND: now also C7.2
- net vdd_mcu: now also C7.1
Changed lines of the file:
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@@
 		(color 0 0 0 0)
 	)
+	(junction
+		(at 140.97 76.2)
+		(diameter 0)
+		(color 0 0 0 0)
+	)
 	(no_connect
 		(at 115.57 118.11)
@@
 	(wire
 		(pts
+			(xy 158.75 76.2) (xy 158.75 82.55)
+		)
+		(stroke
+			(width 0)
+			(type default)
+		)
+	)
+	(wire
+		(pts
 			(xy 106.68 76.2) (xy 106.68 80.01)
 		)
@@
 	(wire
 		(pts
+			(xy 140.97 76.2) (xy 140.97 95.25)
+		)
+		(stroke
+			(width 0)
+			(type default)
+		)
+	)
+	(wire
+		(pts
 			(xy 71.12 46.99) (xy 101.6 46.99)
 		)
@@
 	(wire
 		(pts
-			(xy 140.97 40.64) (xy 140.97 95.25)
+			(xy 140.97 40.64) (xy 140.97 76.2)
 		)
 		(stroke
@@
 		(pts
 			(xy 71.12 40.64) (xy 71.12 46.99)
+		)
+		(stroke
+			(width 0)
+			(type default)
+		)
+	)
+	(wire
+		(pts
+			(xy 158.75 76.2) (xy 140.97 76.2)
 		)
 		(stroke
@@
 		(dnp no)
 		(fields_autoplaced yes)
-		(property "Reference" "#PWR04"
+		(property "Reference" "#PWR09"
 			(at 91.44 113.03 0)
 			(hide yes)
@@
 			(project "sesion2"
 				(path "/d1e9e723-5327-48d1-b5e7-0bbac6992fdf/e7909b8b-0298-42a0-a680-fce37ec3f573"
-					(reference "#PWR04")
+					(reference "#PWR09")
 					(unit 1)
 				)
@@
 		(dnp no)
 		(fields_autoplaced yes)
-		(property "Reference" "R1"
+		(property "Reference" "R2"
 			(at 81.28 88.9 90)
 			(show_name no)
@@
 			)
 		)
-		(property "Footprint" "Package_LCC:PLCC-84_29.3x29.3mm_P1.27mm"
+		(property "Footprint" "Resistor_SMD:R_0402_1005Metric_Pad0.72x0.64mm_HandSolder"
 			(at 81.28 97.028 90)
 			(hide yes)
@@
 			(project "sesion2"
 				(path "/d1e9e723-5327-48d1-b5e7-0bbac6992fdf/e7909b8b-0298-42a0-a680-fce37ec3f573"
-					(reference "R1")
+					(reference "R2")
 					(unit 1)
 				)
@@
 		(dnp no)
 		(fields_autoplaced yes)
-		(property "Reference" "#PWR05"
+		(property "Reference" "#PWR08"
 			(at 83.82 127 0)
 			(hide yes)
@@
 			(project "sesion2"
 				(path "/d1e9e723-5327-48d1-b5e7-0bbac6992fdf/e7909b8b-0298-42a0-a680-fce37ec3f573"
-					(reference "#PWR05")
+					(reference "#PWR08")
+					(unit 1)
+				)
+			)
+		)
+	)
+	(symbol
+		(lib_id "power:GND")
+		(at 158.75 90.17 0)
+		(unit 1)
+		(body_style 1)
+		(exclude_from_sim no)
+		(in_bom yes)
+		(on_board yes)
+		(in_pos_files yes)
+		(dnp no)
+		(fields_autoplaced yes)
+		(property "Reference" "#PWR012"
+			(at 158.75 96.52 0)
+			(hide yes)
+			(show_name no)
+			(do_not_autoplace no)
+			(effects
+				(font
+					(size 1.27 1.27)
+				)
+			)
+		)
+		(property "Value" "GND"
+			(at 158.75 95.25 0)
+			(show_name no)
+			(do_not_autoplace no)
+			(effects
+				(font
+					(size 1.27 1.27)
+				)
+			)
+		)
+		(property "Footprint" "Samacsys:HDRV6W64P0X254_1X6_1524X254X839P"
+			(at 158.75 90.17 0)
+			(hide yes)
+			(show_name no)
+			(do_not_autoplace no)
+			(effects
+				(font
+					(size 1.27 1.27)
+				)
+			)
+		)
+		(property "Datasheet" ""
+			(at 158.75 90.17 0)
+			(hide yes)
+			(show_name no)
+			(do_not_autoplace no)
+			(effects
+				(font
+					(size 1.27 1.27)
+				)
+			)
+		)
+		(property "Description" "Power symbol creates a global label with name \"GND\" , ground"
+			(at 158.75 90.17 0)
+			(hide yes)
+			(show_name no)
+			(do_not_autoplace no)
+			(effects
+				(font
+					(size 1.27 1.27)
+				)
+			)
+		)
+		(pin "1"
+		)
+		(instances
+			(project "sesion2"
+				(path "/d1e9e723-5327-48d1-b5e7-0bbac6992fdf/e7909b8b-0298-42a0-a680-fce37ec3f573"
+					(reference "#PWR012")
 					(unit 1)
 				)
@@
 		(dnp no)
 		(fields_autoplaced yes)
-		(property "Reference" "C3"
+		(property "Reference" "C6"
 			(at 110.49 82.5499 0)
 			(show_name no)
@@
 			)
 		)
-		(property "Footprint" "Samacsys:HDRV6W64P0X254_1X6_1524X254X839P"
+		(property "Footprint" "Capacitor_SMD:C_0402_1005Metric"
 			(at 107.6452 87.63 0)
 			(hide yes)
@@
 			(project "sesion2"
 				(path "/d1e9e723-5327-48d1-b5e7-0bbac6992fdf/e7909b8b-0298-42a0-a680-fce37ec3f573"
-					(reference "C3")
+					(reference "C6")
+					(unit 1)
+				)
+			)
+		)
+	)
+	(symbol
+		(lib_id "Device:C")
+		(at 158.75 86.36 0)
+		(unit 1)
+		(body_style 1)
+		(exclude_from_sim no)
+		(in_bom yes)
+		(on_board yes)
+		(in_pos_files yes)
+		(dnp no)
+		(fields_autoplaced yes)
+		(property "Reference" "C7"
+			(at 162.56 85.0899 0)
+			(show_name no)
+			(do_not_autoplace no)
+			(effects
+				(font
+					(size 1.27 1.27)
+				)
+				(justify left)
+			)
+		)
+		(property "Value" "100nF"
+			(at 162.56 87.6299 0)
+			(show_name no)
+			(do_not_autoplace no)
+			(effects
+				(font
+					(size 1.27 1.27)
+				)
+				(justify left)
+			)
+		)
+		(property "Footprint" "Capacitor_SMD:C_0402_1005Metric"
+			(at 159.7152 90.17 0)
+			(hide yes)
+			(show_name no)
+			(do_not_autoplace no)
+			(effects
+				(font
+					(size 1.27 1.27)
+				)
+			)
+		)
+		(property "Datasheet" ""
+			(at 158.75 86.36 0)
+			(hide yes)
+			(show_name no)
+			(do_not_autoplace no)
+			(effects
+				(font
+					(size 1.27 1.27)
+				)
+			)
+		)
+		(property "Description" "Unpolarized capacitor"
+			(at 158.75 86.36 0)
+			(hide yes)
+			(show_name no)
+			(do_not_autoplace no)
+			(effects
+				(font
+					(size 1.27 1.27)
+				)
+			)
+		)
+		(pin "2"
+		)
+		(pin "1"
+		)
+		(instances
+			(project "sesion2"
+				(path "/d1e9e723-5327-48d1-b5e7-0bbac6992fdf/e7909b8b-0298-42a0-a680-fce37ec3f573"
+					(reference "C7")
 					(unit 1)
 				)
@@
 		(dnp no)
 		(fields_autoplaced yes)
-		(property "Reference" "#PWR02"
+		(property "Reference" "#PWR07"
 			(at 66.04 49.53 0)
 			(hide yes)
@@
 			(project "sesion2"
 				(path "/d1e9e723-5327-48d1-b5e7-0bbac6992fdf/e7909b8b-0298-42a0-a680-fce37ec3f573"
-					(reference "#PWR02")
+					(reference "#PWR07")
 					(unit 1)
 				)
@@
 		(in_pos_files yes)
 		(dnp no)
-		(property "Reference" "J1"
+		(property "Reference" "J2"
 			(at 110.998 39.624 0)
 			(show_name no)
@@
 			(project "sesion2"
 				(path "/d1e9e723-5327-48d1-b5e7-0bbac6992fdf/e7909b8b-0298-42a0-a680-fce37ec3f573"
-					(reference "J1")
+					(reference "J2")
 					(unit 1)
 				)
@@
 		(dnp no)
 		(fields_autoplaced yes)
-		(property "Reference" "#PWR03"
+		(property "Reference" "#PWR010"
 			(at 106.68 93.98 0)
 			(hide yes)
@@
 			(project "sesion2"
 				(path "/d1e9e723-5327-48d1-b5e7-0bbac6992fdf/e7909b8b-0298-42a0-a680-fce37ec3f573"
-					(reference "#PWR03")
+					(reference "#PWR010")
 					(unit 1)
 				)
@@
 		(dnp no)
 		(fields_autoplaced yes)
-		(property "Reference" "C2"
+		(property "Reference" "C4"
 			(at 87.63 115.5699 0)
 			(show_name no)
@@
 			)
 		)
-		(property "Footprint" "Samacsys:HDRV6W64P0X254_1X6_1524X254X839P"
+		(property "Footprint" "Capacitor_SMD:C_0402_1005Metric"
 			(at 84.7852 120.65 0)
 			(hide yes)
@@
 			(project "sesion2"
 				(path "/d1e9e723-5327-48d1-b5e7-0bbac6992fdf/e7909b8b-0298-42a0-a680-fce37ec3f573"
-					(reference "C2")
+					(reference "C4")
 					(unit 1)
 				)
@@
 			)
 		)
-		(property "Footprint" "Package_LCC:PLCC-84_29.3x29.3mm_P1.27mm"
+		(property "Footprint" "Resistor_SMD:R_0402_1005Metric_Pad0.72x0.64mm_HandSolder"
 			(at 96.52 77.978 90)
 			(hide yes)
@@
 		(dnp no)
 		(fields_autoplaced yes)
-		(property "Reference" "R2"
+		(property "Reference" "R1"
 			(at 73.66 102.87 90)
 			(show_name no)
@@
 			)
 		)
-		(property "Footprint" "Package_LCC:PLCC-84_29.3x29.3mm_P1.27mm"
+		(property "Footprint" "Resistor_SMD:R_0402_1005Metric_Pad0.72x0.64mm_HandSolder"
 			(at 73.66 110.998 90)
 			(hide yes)
@@
 			(project "sesion2"
 				(path "/d1e9e723-5327-48d1-b5e7-0bbac6992fdf/e7909b8b-0298-42a0-a680-fce37ec3f573"
-					(reference "R2")
+					(reference "R1")
 					(unit 1)
 				)
@@
 		(dnp no)
 		(fields_autoplaced yes)
-		(property "Reference" "#PWR01"
+		(property "Reference" "#PWR011"
 			(at 135.89 184.15 0)
 			(hide yes)
@@
 			(project "sesion2"
 				(path "/d1e9e723-5327-48d1-b5e7-0bbac6992fdf/e7909b8b-0298-42a0-a680-fce37ec3f573"
-					(reference "#PWR01")
+					(reference "#PWR011")
 					(unit 1)
 				)
@@
 		(dnp no)
 		(fields_autoplaced yes)
-		(property "Reference" "C1"
+		(property "Reference" "C5"
 			(at 95.25 101.5999 0)
 			(show_name no)
@@
 			)
 		)
-		(property "Footprint" "Samacsys:HDRV6W64P0X254_1X6_1524X254X839P"
+		(property "Footprint" "Capacitor_SMD:C_0402_1005Metric"
 			(at 92.4052 106.68 0)
 			(hide yes)
@@
 			(project "sesion2"
 				(path "/d1e9e723-5327-48d1-b5e7-0bbac6992fdf/e7909b8b-0298-42a0-a680-fce37ec3f573"
-					(reference "C1")
+					(reference "C5")
 					(unit 1)
 				)

Commit message: sesion 4
Parts:
- removed C7: 100nF, Capacitor_SMD:C_0402_1005Metric, symbol Device:C
- removed IC1: AT89LS51-16AU, Samacsys:QFP80P1200X1200X120-44N, symbol Samacsys:AT89LS51-16AU
- removed J2: 68000-106HLF, Samacsys:HDRV6W64P0X254_1X6_1524X254X839P, symbol Samacsys:68000-106HLF
- added C4, C9: 100nF, Capacitor_SMD:C_0402_1005Metric, symbol Device:C
- added IC1: PIC16F18855-I_SP, Samacsys:DIP794W56P254L3486H508Q28N, symbol Samacsys:PIC16F18855-I_SP
- added J2, J3: Conn_01x05, Connector_PinHeader_2.54mm:PinHeader_1x05_P2.54mm_Vertical, symbol Connector_Generic:Conn_01x05
- added J5: USB_C_Receptacle_USB2.0_16P, Connector_USB:USB_C_Receptacle_GCT_USB4105-xx-A_16P_TopMnt_Horizontal, symbol Connector:USB_C_Receptacle_USB2.0_16P
- added R10, R9: 5.1k, Resistor_SMD:R_0402_1005Metric_Pad0.72x0.64mm_HandSolder, symbol Device:R
- added R4: 10k, Resistor_SMD:R_0402_1005Metric_Pad0.72x0.64mm_HandSolder, symbol Device:R
- added U2: CH340C, Package_SO:SOIC-16_3.9x9.9mm_P1.27mm, symbol Interface_USB:CH340C
- R1, R2, R3: value 10k -> 1k
- renumbered C4 to C1, C5 to C2, C6 to C3
Connections:
- net GND: now also C4.2, C9.2, IC1.19 (VSS_2), IC1.8 (VSS_1), J2.1 (Pin_1), J3.3 (Pin_3), J5.A1 (GND), J5.A12 (GND), J5.B1 (GND), J5.B12 (GND), J5.SH (SHIELD), R10.1, R9.1, U2.1 (GND)
- net at R2.1: now also J2.3 (Pin_3)
- net at C2.1, R2.2: now also IC1.3 (RA1)
- net at C3.1, R3.2: now also IC1.2 (RA0)
- net at C1.1, R1.2: now also IC1.4 (RA2)
- net at R1.1: now also J2.2 (Pin_2)
- net at R3.1: now also J2.4 (Pin_4)
- new net: J5.A4 (VBUS), J5.A9 (VBUS), J5.B4 (VBUS), J5.B9 (VBUS)
- new net: J5.A5 (CC1), R10.2
- new net: J5.B5 (CC2), R9.2
- new net 3.3v: C4.1, C9.1, IC1.20 (VDD), J2.5 (Pin_5), J3.2 (Pin_2), R4.2, U2.16 (VCC), U2.4 (V3)
- new net DQ: IC1.26 (RB5)
- new net I2C_SCL: IC1.14 (RC3)
- new net I2C_SDA: IC1.15 (RC4)
- new net MCLR/VPP: IC1.1 (VPP/~{MCLR}/RE3), J3.1 (Pin_1), R4.1
- new net PGC: IC1.27 (RB6), J3.4 (Pin_4)
- new net PGD: IC1.28 (RB7), J3.5 (Pin_5)
- new net SPI_CS: IC1.13 (RC2)
- new net SPI_MISO: IC1.12 (RC1)
- new net SPI_SCK: IC1.11 (RC0)
- new net UART_RX: IC1.18 (RC7), U2.3 (RXD)
- new net UART_TX: IC1.17 (RC6), U2.2 (TXD)
- new net USB_D+: J5.A6 (D+), J5.B6 (D+), U2.5 (UD+)
- new net USB_D-: J5.A7 (D-), J5.B7 (D-), U2.6 (UD-)
- new net XHUT: IC1.25 (RB4)
- no-connect marks 40 -> 20
Other:
- moved on the sheet: C1, C2, C3, R1, R2, R3

Commit message: Se han implementado componentes de protección en las líneas de entrada
Parts:
- added D3: D_TVS, Diode_SMD:D_0402_1005Metric, symbol Device:D_TVS
- added D4: D_TVS, Diode_SMD:D_SMA, symbol Device:D_TVS
Connections:
- net 3.3v: now also D3.1 (A1), D4.2 (A2)
- net GND: now also D3.2 (A2), D4.1 (A1)
